Commit message: Examples ready to get time results

File: data/TROmodels/nao_inertial_XYZ_python.urdf (robot description, URDF)
Before this commit: robot nao_inertial_python, 25 links, 24 joints
Joints:
- joint Joint10: axis 1 0 0 -> 0 0 1
- joint Joint11: axis 0 1 0 -> 1 0 0
- joint Joint13: axis 1 0 0 -> 0 1 0
- joint Joint17: axis 0 1 0 -> 0 0 1
- joint Joint18: axis 0 0 1 -> 1 0 0
- joint Joint20: axis 0 1 0 -> 1 0 0
- joint Joint21: axis 0 0 1 -> 0 1 0
- joint Joint22: axis 1 0 0 -> 0 1 0
- joint Joint24: axis 0 0 1 -> 1 0 0
- joint Joint3: axis 0 0 1 -> 0 1 0
- joint Joint4: axis 1 0 0 -> 0 1 0
- joint Joint5: axis 0 1 0 -> 1 0 0
- joint Joint7: axis 1 0 0 -> 0 1 0
- joint Joint8: axis 0 1 0 -> 0 0 1
- joint Joint9: axis 0 0 1 -> 1 0 0
- joint joint6: axis 0 0 1 -> 1 0 0
